Commit message: change convert pipeline,bugs in doors

File: house_7/house_7.urdf (robot description, URDF)
Before this commit: robot house_7, 32 links, 31 joints
Links:
- link AlarmClock_2_3: geometry visual mesh filename=file://house_7/meshes/obj/AlarmClockButton_11.obj scale=1.0 1.0 1.0; visual mesh filename=file://house_7/meshes/obj/AlarmClockButton_11_GeomSubset_0.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 scale=1.0 1.0 1.0
- link ArmChair_2_2_0: geometry visual mesh filename=file://house_7/meshes/obj/Armchair_208.obj scale=1.0 1.0 1.0; visual mesh filename=file://house_7/meshes/obj/Armchair_208_GeomSubset_0.obj scale=1.0 1.0 1.0
- link Chair_2_3_1: geometry visual mesh filename=file://house_7/meshes/obj/Chair_204.obj scale=1.0 1.0 1.0; visual mesh filename=file://house_7/meshes/obj/Chair_204_GeomSubset_0.obj scale=1.0 1.0 1.0
- link Chair_2_3_2: geometry visual mesh filename=file://house_7/meshes/obj/Chair_204.obj scale=1.0 1.0 1.0; visual mesh filename=file://house_7/meshes/obj/Chair_204_GeomSubset_0.obj scale=1.0 1.0 1.0
- link Chair_2_3_3: geometry visual mesh filename=file://house_7/meshes/obj/Chair_204.obj scale=1.0 1.0 1.0; visual mesh filename=file://house_7/meshes/obj/Chair_204_GeomSubset_0.obj scale=1.0 1.0 1.0
- link DiningTable_2_3_0: geometry visual mesh filename=file://house_7/meshes/obj/DiningTable_208.obj scale=1.0 1.0 1.0; visual mesh filename=file://house_7/meshes/obj/DiningTable_208_GeomSubset_0.obj scale=1.0 1.0 1.0
- link Door_0: geometry visual mesh filename=file://house_7/meshes/obj/DoorwayDoor_9.obj scale=1.0 1.0 1.0; visual mesh filename=file://house_7/meshes/obj/DoorwayDoor_9_GeomSubset_0.obj scale=1.0 1.0 1.0
- link Door_1: geometry visual mesh filename=file://house_7/meshes/obj/DoorwayDoor_1.obj scale=1.0 1.0 1.0; visual mesh filename=file://house_7/meshes/obj/DoorwayDoor_1_GeomSubset_0.obj scale=1.0 1.0 1.0
- link FloorLamp_2_2_1: geometry visual mesh filename=file://house_7/meshes/obj/FloorLamp_19.obj scale=1.0 1.0 1.0; visual mesh filename=file://house_7/meshes/obj/FloorLamp_19_GeomSubset_0.obj scale=1.0 1.0 1.0
- link Plunger_3_2: geometry visual mesh filename=file://house_7/meshes/obj/Plunger.obj scale=1.0 1.0 1.0; visual mesh filename=file://house_7/meshes/obj/Plunger_GeomSubset_0.obj scale=1.0 1.0 1.0
- link Sink_3_1_0: geometry visual mesh filename=file://house_7/meshes/obj/PsSinkbasin_15.obj scale=1.0 1.0 1.0; visual mesh filename=file://house_7/meshes/obj/Sink_15.obj scale=1.0 1.0 1.0
- link Statue_2_1: geometry visual mesh filename=file://house_7/meshes/obj/FertilityStatue.obj scale=1.0 1.0 1.0; visual mesh filename=file://house_7/meshes/obj/FertilityStatue_GeomSubset_0.obj scale=1.0 1.0 1.0

Commit message: remove unsplited files

File: house_7/house_7.urdf (robot description, URDF)
Before this commit: robot house_7, 32 links, 31 joints
Links:
- link AlarmClock_2_3: geometry visual mesh filename=file://house_7/meshes/obj/AlarmClockButton_11_AlarmClockBut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 scale=1.0 1.0 1.0; visual mesh filename=file://house_7/meshes/obj/AlarmClockButton_11_AlarmClockBut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 scale=1.0 1.0 1.0
- link ArmChair_2_2_0: geometry visual mesh filename=file://house_7/meshes/obj/Fp208_Armchair3Armchair_208_0_Geo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 scale=1.0 1.0 1.0; visual mesh filename=file://house_7/meshes/obj/Fp208_Armchair3Armchair_208_0_Geo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 scale=1.0 1.0 1.0
- link Bed_2_0_0: geometry visual mesh filename=file://house_7/meshes/obj/BedMattress_1_BedMattress_1_1.obj scale=1.0 1.0 1.0; visual mesh filename=file://house_7/meshes/obj/BedsheetUnmade_1_BedsheetUnmade_1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 scale=1.0 1.0 1.0
- link Chair_2_3_1: geometry visual mesh filename=file://house_7/meshes/obj/ChairmeshChair_204_0_GeomSubset_0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 scale=1.0 1.0 1.0; visual mesh filename=file://house_7/meshes/obj/ChairmeshChair_204_0_GeomSubset_1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 scale=1.0 1.0 1.0
- link Chair_2_3_2: geometry visual mesh filename=file://house_7/meshes/obj/ChairmeshChair_204_0_GeomSubset_0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 scale=1.0 1.0 1.0; visual mesh filename=file://house_7/meshes/obj/ChairmeshChair_204_0_GeomSubset_1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 scale=1.0 1.0 1.0
- link Chair_2_3_3: geometry visual mesh filename=file://house_7/meshes/obj/ChairmeshChair_204_0_GeomSubset_0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 scale=1.0 1.0 1.0; visual mesh filename=file://house_7/meshes/obj/ChairmeshChair_204_0_GeomSubset_1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 scale=1.0 1.0 1.0
- link DiningTable_2_3_0: geometry visual mesh filename=file://house_7/meshes/obj/TablemeshDiningTable_208_0_GeomSu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 scale=1.0 1.0 1.0; visual mesh filename=file://house_7/meshes/obj/TablemeshDiningTable_208_0_GeomSu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 scale=1.0 1.0 1.0
- link Door_0: geometry visual mesh filename=file://house_7/meshes/obj/MeshDoorwayDoor_9_0_GeomSubset_0.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 scale=1.0 1.0 1.0; visual mesh filename=file://house_7/meshes/obj/MeshDoorwayDoor_9_0_GeomSubset_1.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 scale=1.0 1.0 1.0
- link Door_1: geometry visual mesh filename=file://house_7/meshes/obj/MeshDoorwayDoor_1_1_GeomSubset_0.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 scale=1.0 1.0 1.0; visual mesh filename=file://house_7/meshes/obj/MeshDoorwayDoor_1_1_GeomSubset_1.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 scale=1.0 1.0 1.0
- link Dresser_2_1: geometry visual mesh filename=file://house_7/meshes/obj/DrawermeshDresserDrawer_229_1_1.o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 scale=1.0 1.0 1.0; visual mesh filename=file://house_7/meshes/obj/DrawermeshDresserDrawer_229_2_2.o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 scale=1.0 1.0 1.0
- link Faucet_3_1_1: geometry visual mesh filename=file://house_7/meshes/obj/MeshSinkFaucet_19_0.obj scale=1.0 1.0 1.0; visual mesh filename=file://house_7/meshes/obj/SinkFaucetKnob_19_SinkFaucetKnob_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 scale=1.0 1.0 1.0
- link FloorLamp_2_2_1: geometry visual mesh filename=file://house_7/meshes/obj/MeshFloorLamp_19_0_GeomSubset_0.o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 scale=1.0 1.0 1.0; visual mesh filename=file://house_7/meshes/obj/MeshFloorLamp_19_0_GeomSubset_1.o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 scale=1.0 1.0 1.0
- link Pillow_2_0_1: geometry visual mesh filename=file://house_7/meshes/obj/MeshPillow_13_0.obj scale=1.0 1.0 1.0
- link Plunger_3_2: geometry visual mesh filename=file://house_7/meshes/obj/MeshPlunger_0_GeomSubset_0.obj scale=1.0 1.0 1.0; visual mesh filename=file://house_7/meshes/obj/MeshPlunger_0_GeomSubset_1.obj scale=1.0 1.0 1.0
- link Sink_3_1_0: geometry visual mesh filename=file://house_7/meshes/obj/MeshPsSinkbasin_15_1.obj scale=1.0 1.0 1.0; visual mesh filename=file://house_7/meshes/obj/Sink_15_Sink_15_0_GeomSubset_0.obj scale=1.0 1.0 1.0
- link Statue_2_1: geometry visual mesh filename=file://house_7/meshes/obj/MeshFertilityStatue_0_GeomSubset_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 scale=1.0 1.0 1.0; visual mesh filename=file://house_7/meshes/obj/MeshFertilityStatue_0_GeomSubset_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 scale=1.0 1.0 1.0
- link ToiletPaper_3_4: geometry visual mesh filename=file://house_7/meshes/obj/PaperToiletpaper_1.obj scale=1.0 1.0 1.0; visual mesh filename=file://house_7/meshes/obj/RollRoll_0.obj scale=1.0 1.0 1.0
- link Toilet_3_0: geometry visual mesh filename=file://house_7/meshes/obj/Fp401_ToiletlidmeshFp401_Toiletli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 scale=1.0 1.0 1.0; visual mesh filename=file://house_7/meshes/obj/MeshFp401_Toiletbody_0.obj scale=1.0 1.0 1.0
- link Vase_2_0: geometry visual mesh filename=file://house_7/meshes/obj/MeshVaseTall_0.obj scale=1.0 1.0 1.0

Commit message: better implementation for walls and windows

File: house_7/house_7.urdf (robot description, URDF)
Before this commit: robot house_7, 32 links, 31 joints
Links:
- removed link Wall_11
- added link Wall_9; visual mesh filename=file://house_7/meshes/stl/Wall_9.stl scale=1.0 1.0 1.0
- added link Window_0; visual mesh filename=file://house_7/meshes/obj/MeshWindowFixed_60X72_0_GeomSubse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 scale=1.0 1.0 1.0; visual mesh filename=file://house_7/meshes/obj/MeshWindowFixed_60X72_0_GeomSubse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 scale=1.0 1.0 1.0
- added link Window_1; visual mesh filename=file://house_7/meshes/obj/MeshWindowHung_44X60_0_GeomSubset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 scale=1.0 1.0 1.0; visual mesh filename=file://house_7/meshes/obj/MeshWindowHung_44X60_0_GeomSubset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 scale=1.0 1.0 1.0
- link Wall_1: geometry visual mesh filename=file://house_7/meshes/stl/Wall_1_0.stl scale=1.0 1.0 1.0; visual mesh filename=file://house_7/meshes/stl/Wall_1_1.stl scale=1.0 1.0 1.0
- link Wall_3: geometry visual mesh filename=file://house_7/meshes/stl/Wall_3_0.stl scale=1.0 1.0 1.0; visual mesh filename=file://house_7/meshes/stl/Wall_3_1.stl scale=1.0 1.0 1.0
Joints:
- removed joint Wall_11_joint
- added joint Wall_9_joint: type fixed, parent house_7, child Wall_9, origin xyz=0.0 0.0 0.0 rpy=1.5707963705062866 0.0 0.0
- added joint Window_0_joint: type fixed, parent house_7, child Window_0, origin xyz=8.245738943496418 -10.123 1.3084695730051197 rpy=0.0 0.0 0.0
- added joint Window_1_joint: type fixed, parent house_7, child Window_1, origin xyz=5.276376266351104 -8.098 1.3099458012422718 rpy=0.0 0.0 0.0
