Commit message: fix different scale units

File: house_5/house_5.urdf (robot description, URDF)
Before this commit: robot house_5, 89 links, 88 joints
Links:
- removed link Wall_18
- removed link Wall_19
- removed link Wall_20
- removed link Wall_21
- removed link Wall_24
- removed link Wall_25
- added link Wall_14; visual mesh filename=file://house_5/meshes/stl/Wall_14.stl scale=1.0 1.0 1.0
- added link Wall_15; visual mesh filename=file://house_5/meshes/stl/Wall_15.stl scale=1.0 1.0 1.0
- added link Wall_16; visual mesh filename=file://house_5/meshes/stl/Wall_16_0.stl scale=1.0 1.0 1.0; visual mesh filename=file://house_5/meshes/stl/Wall_16_1.stl scale=1.0 1.0 1.0
- added link Wall_9; visual mesh filename=file://house_5/meshes/stl/Wall_9.stl scale=1.0 1.0 1.0
- added link Window_0; visual mesh filename=file://house_5/meshes/obj/MeshWindowBay_2_0_GeomSubset_0.obj scale=1.0 1.0 1.0; visual mesh filename=file://house_5/meshes/obj/MeshWindowBay_2_0_GeomSubset_1.obj scale=1.0 1.0 1.0
- link Wall_4: geometry visual mesh filename=file://house_5/meshes/stl/Wall_4_0.stl scale=1.0 1.0 1.0; visual mesh filename=file://house_5/meshes/stl/Wall_4_1.stl scale=1.0 1.0 1.0
Joints:
- removed joint Wall_18_joint
- removed joint Wall_19_joint
- removed joint Wall_20_joint
- removed joint Wall_21_joint
- removed joint Wall_24_joint
- removed joint Wall_25_joint
- added joint Wall_14_joint: type fixed, parent house_5, child Wall_14, origin xyz=0.0 0.0 0.0 rpy=1.5707963705062866 0.0 0.0
- added joint Wall_15_joint: type fixed, parent house_5, child Wall_15, origin xyz=0.0 0.0 0.0 rpy=1.5707963705062866 0.0 0.0
- added joint Wall_16_joint: type fixed, parent house_5, child Wall_16, origin xyz=0.0 0.0 0.0 rpy=1.5707963705062866 0.0 0.0
- added joint Wall_9_joint: type fixed, parent house_5, child Wall_9, origin xyz=0.0 0.0 0.0 rpy=1.5707963705062866 0.0 0.0
- added joint Window_0_joint: type fixed, parent house_5, child Window_0, origin xyz=8.374918929768196 0.0 1.3006609899632153 rpy=0.0 0.0 0.0
